File: PCB/analog_section.kicad_sch (KiCad schematic)
At the start: 86 parts, among them J3 Probe +, J4 Probe +, J5 Probe -, J6 Probe -, K1 G6K-2, K2 G6K-2, K3 G6K-2, Q1 NMOS, Q2 NMOS, Q3 NMOS, U1 TLV757P, U3 AD9833xRM, U4 LMH6643MMX, U6 LMH6643MMX, U7 LMH6643MMX, Y1 25MHz

Commit message: Changed opamps
Changed opamps to OPA2197, which has higher open loop gain and much
lower GBW. This opamp should be much more forgiving of parasitic
capacitance and hopefully solve the ringing issue.

Also fixed MOSFET orientation issue which has plagued this design until
now, no wonder the BPS didn't work.

Additionally changed firmware to use the new version of the button
debouncing module from the embedded_c_modules repo.
Parts:
- removed Q1, Q2, Q3: NMOS, Package_TO_SOT_SMD:SOT-23-3, symbol Simulation_SPICE:NMOS
- removed U4, U6, U7: LMH6643MMX, CustomFootprints:VSSOP-8_3x3mm_P0.65mm, symbol Device:Opamp_Dual
- added Q1, Q2, Q3: NMOS, Package_TO_SOT_SMD:SOT-23, symbol Transistor_FET:2N7002
- added U4, U6, U7: OPA2197xDGK, CustomFootprints:VSSOP-8_3x3mm_P0.65mm, symbol Amplifier_Operational:OPA2197xDGK
- J3, J4: footprint Connector:Banana_Cliff_FCR7350R_S16N-PC_Horizontal -> CustomFootprints:Banana_Red
- J5, J6: footprint Connector:Banana_Cliff_FCR7350B_S16N-PC_Horizontal -> CustomFootprints:Banana_Black
- renumbered C14 to C13, C19 to C16, C20 to C17, C22 to C18, C23 to C19, C24 to C20, C32 to C30, R9 to R10, R11 to R12, R12 to R13, R13 to R15, R15 to R18, R1 to R2, R17 to R20, R18 to R21, R20 to R23, R21 to R24, R22 to R25, R23 to R26, R24 to R27, R25 to R28, R26 to R29, R27 to R30, R28 to R31, R29 to R32, R30 to R33, R2 to R4, R3 to R6, R4 to R7, R6 to R8, R7 to R9
Connections:
- net +3V3A: now also U4.8 (V+), U6.8 (V+)
- net +5V: now also U7.8 (V+)
- net -3V3A: now also U4.4 (V-), U6.4 (V-), U7.4 (V-)
- net COIL_D1: now also Q1.3 (D)
- net COIL_D2: now also Q2.3 (D)
- net COIL_D3: now also Q3.3 (D)
- net COIL_G1: now also Q1.1 (G)
- net COIL_G2: now also Q2.1 (G)
- net COIL_G3: now also Q3.1 (G)
- net DDS_HPF: now also U4.5 (+)
- net DDS_LPF_1: now also U4.3 (+)
- net DDS_LPF_2: now also U4.1, U4.2 (-)
- net GND: now also Q1.2 (S), Q2.2 (S), Q3.2 (S), U6.3 (+), U6.5 (+)
- net INV: now also U4.6 (-)
- net RANGE_1_P1: now also U4.7
- net RANGE_2_P1: now also U6.2 (-)
- net RANGE_2_P2: now also U6.1
- net RANGE_3_P1: now also U6.6 (-)
- net RANGE_3_P2: now also U6.7
- net dut_curr_2: now also U7.5 (+)
- net dut_curr_3: now also U7.6 (-), U7.7
- net dut_test_2: now also U7.3 (+)
- net dut_test_3: now also U7.1, U7.2 (-)
