File: PCB/analog_section.kicad_sch (KiCad schematic)
At the start: 86 parts, among them J3 Probe +, J4 Probe +, J5 Probe -, J6 Probe -, K1 G6K-2, K2 G6K-2, K3 G6K-2, Q1 NMOS, Q2 NMOS, Q3 NMOS, U1 TLV757P, U3 AD9833xRM, U4 OPA2197xDGK, U6 OPA2197xDGK, U7 OPA2197xDGK, Y1 25MHz

Commit message: Added soft-start
Also added new case step files
Parts:
- renumbered C1 to C25, C2 to C26, C3 to C27, C4 to C28, C5 to C29, C13 to C30, C16 to C31, C17 to C32, C18 to C33, C19 to C34, C20 to C35, C30 to C36, C33 to C37, C34 to C38, C35 to C39, C36 to C40, C37 to C41, C38 to C42, C39 to C43, C40 to C44, D9 to D10, D1 to D2, D2 to D3, D3 to D4, D4 to D5, D5 to D6, D6 to D7, D7 to D8, D8 to D9, R2 to R11, R4 to R12, R6 to R13, R7 to R14, R8 to R15, R9 to R16, R10 to R17, R12 to R18, R13 to R19, R15 to R20, R18 to R21, R20 to R22, R21 to R23, R23 to R24, R24 to R25, R25 to R26, R26 to R27, R27 to R28, R28 to R29, R29 to R30, R30 to R31, R31 to R32, R32 to R33, R33 to R34, TP6 to TP10, TP7 to TP11, TP8 to TP12, TP11 to TP13, TP12 to TP14, TP13 to TP15, TP14 to TP16, TP15 to TP17, TP1 to TP5, TP2 to TP6, TP3 to TP7, TP4 to TP8, TP5 to TP9, U7 to U10, U1 to U6, U3 to U7, U4 to U8, U6 to U9, Y1 to Y2
