File: PCB/lcr.kicad_sch (KiCad schematic)
At the start: 48 parts, among them J1 Conn_01x04_Pin, J2 USB_C_Receptacle_USB2.0_14P, SW1 SW_Push, SW2 SW_Push, U2 UMW HT7836-A, U5 STM32G431CBT6, U8 TLV757P, U9 USBLC6-2SC6, Y2 8 MHz

Commit message: Changed opamps
Changed opamps to OPA2197, which has higher open loop gain and much
lower GBW. This opamp should be much more forgiving of parasitic
capacitance and hopefully solve the ringing issue.

Also fixed MOSFET orientation issue which has plagued this design until
now, no wonder the BPS didn't work.

Additionally changed firmware to use the new version of the button
debouncing module from the embedded_c_modules repo.
Parts:
- removed C17, C18: 10u, Capacitor_SMD:C_0603_1608Metric, symbol Device:C
- removed U2: UMW HT7836-A, Package_TO_SOT_SMD:SOT-89-3, symbol Regulator_Linear:MCP1703Ax-400xxMB
- added C14, C15: 10u, Capacitor_SMD:C_0603_1608Metric, symbol Device:C
- added R1: 5k1, Resistor_SMD:R_0603_1608Metric, symbol Device:R
- added R3, R5: 1k, Resistor_SMD:R_0603_1608Metric, symbol Device:R
- added U2: TLV75801PDBV, Package_TO_SOT_SMD:SOT-23-5, symbol Regulator_Linear:TLV75801PDBV
- renumbered C11 to C10, C12 to C11, C13 to C12, C25 to C21, C26 to C22, C27 to C23, C6 to C24, C15 to C25, C16 to C26, C29 to C27, C30 to C28, C21 to C29, C28 to C31, C31 to C32, C7 to C6, C8 to C7, C9 to C8, C10 to C9, R10 to R11, R5 to R14, R8 to R16, R14 to R17, R16 to R19, R19 to R22
Connections:
- net +5V: now also C14.2, U2.1 (IN), U2.3 (EN)
- net GND: now also C14.1, C15.1, R5.1, U2.2 (GND)
- net +3V6 renamed +3V9
- net +3V9: now also C15.2, R1.2, U2.5 (OUT)
- new net: R1.1, R3.2
- new net 3V9FB: R3.1, R5.2, U2.4 (FB)
Other:
- note added: "VOUT = VFB × (1 + R1 / R2) VOUT = 0.55 × (1 + 6.1 / 1) = 3.905V"
- moved on the sheet: C24, C25, C26, C29, C31, C32, DS1, H1, H2, H3, H4, R14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
